File: MICRO-ROUTER-PCB/MICRO-ROUTER/MICRO-ROUTER.kicad_pcb (KiCad board)
At the start: 2 copper layers, 85 x 54 mm, 79 parts, among them J2 USB_A, J3 USB_C_Receptacle_USB2.0_16P, J4 Battery Connector, J5 SPI Header, J6 GPIO Header, J7 RJ45 5-2301996-6, Q1 FS8205A, SW2 8Devices Reset, SW3 UART Reset, U1 TP4056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

Commit message: -Unrouted PCB Errors
Parts:
- added C22: 0.1uf, Capacitor_SMD:C_0603_1608Metric, F.Cu at (153.4, 151.5)
- added C9: 4.7uf, Capacitor_SMD:C_0603_1608Metric, F.Cu at (146.5, 153.8)
- added D5: LED, LED_SMD:LED_0603_1608Metric, F.Cu at (157.5, 149.0)
- added D6: LED, LED_SMD:LED_0603_1608Metric, F.Cu at (157.5, 151.6)
- added D8: SP0503BAHT, Package_TO_SOT_SMD:SOT-143, F.Cu at (143.5, 141.3)
- added R11: 75Ω, Resistor_SMD:R_0603_1608Metric, F.Cu at (153.4, 154.0)
- added R12: 75Ω, Resistor_SMD:R_0603_1608Metric, F.Cu at (153.4, 156.5)
- added R27: 1K, Resistor_SMD:R_0603_1608Metric_Pad0.98x0.95mm_HandSolder, F.Cu at (157.6, 158.8)
- J4: value Battery Connector -> Battery Connector
- U2: value XC9142B33DMR-G -> XC9142B33DMR-G
Connections:
- U3 pad 15: CTS -> RTS
- U3 pad 16: RTS -> CTS
- U3 pad 19: Net-(U3-~{RXT}/GPIO.3) -> Net-(D6-K)
- U3 pad 20: Net-(U3-~{TXT}/GPIO.2) -> Net-(D5-K)
- U3 pad 6: unconnected-(U3-VDD-Pad6) -> +3.3V
Routing:
- net Net-(U3-~{RST}): track 82.8 -> 6.50 mm, vias 1 -> 0
- net +3.3V: track 161.5 -> 99.5 mm, vias 6 -> 4
- net RTS: track 41.4 -> 0.00 mm, vias 1 -> 0
- net CTS: track 41.2 -> 0.00 mm, vias 1 -> 0
- net Net-(U3-~{RXT}/GPIO.3): track 11.4 -> 0.00 mm
- net VBUS: track 21.2 -> 10.2 mm
- net Net-(U3-~{TXT}/GPIO.2): track 9.69 -> 0.00 mm
- net Net-(U3-TXD): track 8.73 -> 0.00 mm
- net Net-(U3-RXD): track 6.17 -> 0.00 mm
- net USB-C-D+: track 8.35 -> 6.36 mm
- net USB-C-D-: track 8.13 -> 6.15 mm
- net GND: track 32.3 -> 31.3 mm, vias 206 -> 205

Commit message: -Fixed the ttl adapter (this time should be right)
Parts:
- removed the D5 at (157.5, 149.0)
- removed the D5 at (127.5, 135.0)
- removed the D6 at (127.5, 137.8)
- removed the D6 at (157.5, 151.6)
- removed the R11 at (153.4, 154.0)
- removed the R11 at (131.8, 148.5)
- removed the R12 at (153.4, 156.5)
- removed the R12 at (131.7, 146.5)
- removed SW3: UART Reset, Button_Switch_THT:SW_PUSH_6mm
- added D5: LED, LED_SMD:LED_0603_1608Metric, F.Cu at (127.9, 139.5)
- added D6: LED, LED_SMD:LED_0603_1608Metric, F.Cu at (130.5, 141.7)
- added R11: 75Ω, Resistor_SMD:R_0603_1608Metric, F.Cu at (133.0, 142.8)
- added R12: 75Ω, Resistor_SMD:R_0603_1608Metric, F.Cu at (133.0, 141.0)
- moved R27 27.7 mm to (132.9, 146.1), turned to 180 degrees
- moved D8 24.4 mm to (119.2, 143.8)
- moved C22 20.7 mm to (133.0, 147.8), turned to 180 degrees
- moved C9 16.4 mm to (133.0, 144.5), turned to 180 degrees
- moved U3 6.63 mm to (127.8, 146.2), turned to 0 degrees
- moved R3 1.85 mm to (127.9, 141.2)
Routing:
- net +3.3V: track 99.5 -> 156.4 mm, vias 4 -> 5
- net RTS: track 0.00 -> 49.8 mm, vias 0 -> 1
- net CTS: track 0.00 -> 48.3 mm, vias 0 -> 1
- net VBUS: track 10.2 -> 39.0 mm, vias 0 -> 2
- net USB-C-D-: track 6.15 -> 19.1 mm
- net USB-C-D+: track 6.36 -> 19.3 mm
- net Net-(U3-RXD): track 0.00 -> 12.8 mm, vias 0 -> 2
- net Net-(U3-TXD): track 0.00 -> 12.1 mm, vias 0 -> 2
- net Net-(D5-K): track 16.3 -> 6.06 mm
- net Net-(D6-K): track 14.6 -> 6.12 mm
- net Net-(D5-A): track 0.00 -> 7.41 mm
- net GND: track 31.3 -> 36.8 mm, vias 205 -> 218
- net Net-(D6-A): track 0.00 -> 2.63 mm
- net Net-(J3-CC1): track 5.81 -> 6.15 mm, vias 0 -> 2
Other:
- outline, holes or cut-outs redrawn

Commit message: backup before wipe
Parts:
- removed C22: 0.1uf, Capacitor_SMD:C_0603_1608Metric
- removed C9: 4.7uf, Capacitor_SMD:C_0603_1608Metric
- added C23: 4.7uf, Capacitor_SMD:C_0603_1608Metric_Pad1.08x0.95mm_HandSolder, F.Cu at (124.9, 147.0)
- added C24: 0.1uf, Capacitor_SMD:C_0603_1608Metric_Pad1.08x0.95mm_HandSolder, F.Cu at (122.0, 148.1)
- added C25: 0.1uf, Capacitor_SMD:C_0603_1608Metric_Pad1.08x0.95mm_HandSolder, F.Cu at (128.5, 148.8)
- added C26: 4.7uf, Capacitor_SMD:C_0603_1608Metric_Pad1.08x0.95mm_HandSolder, F.Cu at (128.5, 147.0)
- added R28: 22.1k, Resistor_SMD:R_0603_1608Metric, F.Cu at (119.5, 148.0)
- added R29: 47.5k, Resistor_SMD:R_0603_1608Metric, F.Cu at (128.7, 144.8)
- R27: value 1K -> R; footprint Resistor_SMD:R_0603_1608Metric_Pad0.98x0.95mm_HandSolder -> Resistor_SMD:R_0603_1608Metric
- moved R12 5.22 mm to (133.2, 146.2), turned to 90 degrees
- moved R27 5.19 mm to (128.8, 143.0), turned to 0 degrees
- moved D5 4.94 mm to (131.5, 142.9), turned to -90 degrees
- moved U3 4.41 mm to (124.3, 143.5)
- moved R3 3.77 mm to (127.1, 137.6), turned to 90 degrees
- moved R11 3.71 mm to (131.5, 146.1), turned to 90 degrees
- moved R23 3.36 mm to (119.0, 146.5)
- moved R24 3.36 mm to (119.0, 145.0)
- moved D6 2.99 mm to (133.2, 142.9)
- moved R7 1.91 mm to (112.0, 140.5)
- moved C3 1.41 mm to (113.9, 137.3)
- moved R2 1.41 mm to (114.0, 135.3)
- moved D8 1.41 mm to (119.2, 142.3)
- moved J3 1.41 mm to (121.0, 134.0)
- moved R4 1.41 mm to (115.5, 141.6)
Connections:
- R11 pad 1: +3.3V -> IR 3.3v
- R12 pad 1: +3.3V -> IR 3.3v
- R27 pad 1: +3.3V -> Net-(U3-~{RST})
- R27 pad 2: Net-(U3-~{RST}) -> IR 3.3v
- U3 pad 6: +3.3V -> IR 3.3v
- U3 pad 7: +3.3V -> VBUS
- U3 pad 8: VBUS -> Net-(U3-VBUS)
Routing:
- net +3.3V: track 156.4 -> 99.5 mm, vias 5 -> 4
- net IR 3.3v: track 0.00 -> 19.4 mm, vias 0 -> 2
- net RTS: track 49.8 -> 42.4 mm
- net URAT-TX: track 83.7 -> 76.4 mm
- net USB-C-D-: track 19.1 -> 13.3 mm
- net Net-(D5-A): track 7.41 -> 1.64 mm
- net VBUS: track 39.0 -> 33.4 mm, vias 2 -> 0
- net Net-(U3-VBUS): track 0.00 -> 5.52 mm
- net CTS: track 48.3 -> 43.1 mm, vias 1 -> 2
- net URAT-RX: track 80.8 -> 75.9 mm
- net Net-(D5-K): track 6.06 -> 10.9 mm, vias 0 -> 1
- net Net-(D6-K): track 6.12 -> 10.9 mm
- net Net-(U3-TXD): track 12.1 -> 8.14 mm
- net Net-(U3-RXD): track 12.8 -> 8.98 mm
- net GND: track 36.8 -> 33.8 mm, vias 218 -> 211
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