File: MICRO-ROUTER-PCB/MICRO-ROUTER/_autosave-MICRO-ROUTER.kicad_sch (KiCad schematic)
At the start: 80 parts, among them J2 USB_A, J3 USB_C_Receptacle_USB2.0_16P, J4 Battery Connector, J5 SPI Header, J6 GPIO Header, J7 RJ45 5-2301996-6, Q1 FS8205A, SW2 8Devices Reset, U1 TP4056, U2 XC9142B33DMR-G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

Commit message: backup before wipe
Parts:
- R27, R28, R29: footprint Resistor_SMD:R_0201_0603Metric_Pad0.64x0.40mm_HandSolder -> Resistor_SMD:R_0603_1608Metric
Connections:
- net IR 3.3v: now also R11.1, R12.1
Changed lines of the file:
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@@
 	(global_label "IR 3.3v"
 		(shape input)
-		(at 388.62 118.11 0)
+		(at 387.35 118.11 0)
 		(fields_autoplaced yes)
 		(effects
@@
 		)
 		(property "Intersheetrefs" "${INTERSHEET_REFS}"
-			(at 398.439 118.11 0)
+			(at 397.169 118.11 0)
 			(effects
 				(font
@@
 		(shape input)
 		(at 245.11 52.07 0)
-		(fields_autoplaced yes)
 		(effects
 			(font
@@
 			)
 		)
-		(property "Footprint" "Resistor_SMD:R_0201_0603Metric_Pad0.64x0.40mm_HandSolder"
+		(property "Footprint" "Resistor_SMD:R_0603_1608Metric"
 			(at 311.912 86.36 90)
 			(effects
@@
 			)
 		)
-		(property "Footprint" "Resistor_SMD:R_0201_0603Metric_Pad0.64x0.40mm_HandSolder"
+		(property "Footprint" "Resistor_SMD:R_0603_1608Metric"
 			(at 311.912 104.14 90)
 			(effects
@@
 			)
 		)
-		(property "Footprint" "Resistor_SMD:R_0201_0603Metric_Pad0.64x0.40mm_HandSolder"
+		(property "Footprint" "Resistor_SMD:R_0603_1608Metric"
 			(at 339.09 78.232 90)
 			(effects
